File: anet-fan-light/fan_light_module.sch (EAGLE design)
At the start: 8 parts, among them X1 IN-12V, X2 NOZ-FAN, X3 LIGHT, X4 BLK-FAN

Commit message: new projects
Parts:
- added H1: MOUNT-PAD-ROUND3.0, holes:MOUNT-PAD-ROUND3.0
- X4: value BLK-FAN -> EXT-FAN
Other:
- moved on the sheet: JP2, JP3, R1, X3-1, X3-2, X4-1, X4-2
Changed lines of the file:
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@@
 <part name="P+3" library="supply1" deviceset="+12V" device=""/>
 <part name="GND3" library="supply1" deviceset="GND" device=""/>
-<part name="X4" library="Rembrandt Electronics - JST XH Connectors v1-0" deviceset="JST-XH-02-PIN" device="-LONG-PAD" value="BLK-FAN"/>
+<part name="X4" library="Rembrandt Electronics - JST XH Connectors v1-0" deviceset="JST-XH-02-PIN" device="-LONG-PAD" value="EXT-FAN"/>
 <part name="JP3" library="pinhead" deviceset="PINHD-1X2" device=""/>
 <part name="P+4" library="supply1" deviceset="+12V" device=""/>
 <part name="GND4" library="supply1" deviceset="GND" device=""/>
 <part name="R1" library="rcl" deviceset="R-EU_" device="0204/7"/>
+<part name="H1" library="holes" deviceset="MOUNT-PAD-ROUND" device="3.0"/>
 </parts>
 <sheets>
@@
 <instance part="P+2" gate="1" x="50.8" y="60.96"/>
 <instance part="GND2" gate="1" x="50.8" y="45.72"/>
-<instance part="X3" gate="-2" x="76.2" y="50.8" rot="MR0"/>
-<instance part="X3" gate="-1" x="76.2" y="53.34" rot="MR0"/>
-<instance part="JP2" gate="G$1" x="91.44" y="53.34"/>
-<instance part="P+3" gate="1" x="81.28" y="60.96"/>
-<instance part="GND3" gate="1" x="81.28" y="45.72"/>
-<instance part="X4" gate="-2" x="106.68" y="50.8" rot="MR0"/>
-<instance part="X4" gate="-1" x="106.68" y="53.34" rot="MR0"/>
-<instance part="JP3" gate="G$1" x="129.54" y="53.34"/>
-<instance part="P+4" gate="1" x="111.76" y="60.96"/>
-<instance part="GND4" gate="1" x="111.76" y="45.72"/>
-<instance part="R1" gate="G$1" x="116.84" y="53.34"/>
+<instance part="X3" gate="-2" x="7.62" y="25.4" rot="MR0"/>
+<instance part="X3" gate="-1" x="7.62" y="27.94" rot="MR0"/>
+<instance part="JP2" gate="G$1" x="22.86" y="27.94"/>
+<instance part="P+3" gate="1" x="12.7" y="35.56"/>
+<instance part="GND3" gate="1" x="12.7" y="20.32"/>
+<instance part="X4" gate="-2" x="38.1" y="25.4" rot="MR0"/>
+<instance part="X4" gate="-1" x="38.1" y="27.94" rot="MR0"/>
+<instance part="JP3" gate="G$1" x="60.96" y="27.94"/>
+<instance part="P+4" gate="1" x="43.18" y="35.56"/>
+<instance part="GND4" gate="1" x="43.18" y="20.32"/>
+<instance part="R1" gate="G$1" x="48.26" y="27.94"/>
+<instance part="H1" gate="G$1" x="10.16" y="53.34" rot="R90"/>
 </instances>
 <busses>
@@
 <pinref part="X3" gate="-2" pin="S"/>
 <pinref part="GND3" gate="1" pin="GND"/>
-<wire x1="78.74" y1="50.8" x2="81.28" y2="50.8" width="0.1524" layer="91"/>
-<wire x1="81.28" y1="50.8" x2="81.28" y2="48.26" width="0.1524" layer="91"/>
+<wire x1="10.16" y1="25.4" x2="12.7" y2="25.4" width="0.1524" layer="91"/>
+<wire x1="12.7" y1="25.4" x2="12.7" y2="22.86" width="0.1524" layer="91"/>
 </segment>
 <segment>
 <pinref part="X4" gate="-2" pin="S"/>
 <pinref part="GND4" gate="1" pin="GND"/>
-<wire x1="109.22" y1="50.8" x2="111.76" y2="50.8" width="0.1524" layer="91"/>
-<wire x1="111.76" y1="50.8" x2="111.76" y2="48.26" width="0.1524" layer="91"/>
+<wire x1="40.64" y1="25.4" x2="43.18" y2="25.4" width="0.1524" layer="91"/>
+<wire x1="43.18" y1="25.4" x2="43.18" y2="22.86" width="0.1524" layer="91"/>
 </segment>
 </net>
@@
 <segment>
 <pinref part="P+3" gate="1" pin="+12V"/>
-<wire x1="81.28" y1="58.42" x2="81.28" y2="55.88" width="0.1524" layer="91"/>
+<wire x1="12.7" y1="33.02" x2="12.7" y2="30.48" width="0.1524" layer="91"/>
 <pinref part="JP2" gate="G$1" pin="1"/>
-<wire x1="81.28" y1="55.88" x2="88.9" y2="55.88" width="0.1524" layer="91"/>
+<wire x1="12.7" y1="30.48" x2="20.32" y2="30.48" width="0.1524" layer="91"/>
 </segment>
 <segment>
 <pinref part="P+4" gate="1" pin="+12V"/>
-<wire x1="111.76" y1="58.42" x2="111.76" y2="55.88" width="0.1524" layer="91"/>
+<wire x1="43.18" y1="33.02" x2="43.18" y2="30.48" width="0.1524" layer="91"/>
 <pinref part="JP3" gate="G$1" pin="1"/>
-<wire x1="111.76" y1="55.88" x2="127" y2="55.88" width="0.1524" layer="91"/>
+<wire x1="43.18" y1="30.48" x2="58.42" y2="30.48" width="0.1524" layer="91"/>
 </segment>
 </net>
@@
 <pinref part="JP2" gate="G$1" pin="2"/>
 <pinref part="X3" gate="-1" pin="S"/>
-<wire x1="88.9" y1="53.34" x2="78.74" y2="53.34" width="0.1524" layer="91"/>
+<wire x1="20.32" y1="27.94" x2="10.16" y2="27.94" width="0.1524" layer="91"/>
 </segment>
 </net>
@@
 <pinref part="X4" gate="-1" pin="S"/>
 <pinref part="R1" gate="G$1" pin="1"/>
-<wire x1="111.76" y1="53.34" x2="109.22" y2="53.34" width="0.1524" layer="91"/>
+<wire x1="43.18" y1="27.94" x2="40.64" y2="27.94" width="0.1524" layer="91"/>
 </segment>
 </net>
@@
 <pinref part="R1" gate="G$1" pin="2"/>
 <pinref part="JP3" gate="G$1" pin="2"/>
-<wire x1="127" y1="53.34" x2="121.92" y2="53.34" width="0.1524" layer="91"/>
+<wire x1="58.42" y1="27.94" x2="53.34" y2="27.94" width="0.1524" layer="91"/>
 </segment>
 </net>
