File: stellarcore/untitled.brd (EAGLE design)
At the start: 160 x 100 mm, 77 parts, among them Q3 IRF540, Q4 IRF540, Q5 IRF540, Q6 IRF540, X1 04-JST-B4B-XH-A, X10 04-JST-B4B-XH-A, X11 04-JST-B4B-XH-A, X12 04-JST-B4B-XH-A, X13 04-JST-B4B-XH-A, X14 04-JST-B4B-XH-A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

Commit message: new projects
Parts:
- removed C11: (no value), rcl:E2,5-5
- removed C6, C7: (no value), rcl:E2,5-7
- removed JP6, JP7: (no value), jumper:JP3Q
- removed Q3: IRF540, transistor-fet:TO220
- removed R6, R7, R8: (no value), rcl:0204/7
- removed U$16: 03-JST-B3B-XH-A, bt_con-jst-xh:B3B-XH
- removed X11, X12, X13, X14, X16, X6, X7, X8, X9: 04-JST-B4B-XH-A, bt_con-jst-xh:B4B-XH
- added U$12: 03-JST-B3B-XH-A, bt_con-jst-xh:B3B-XH
- U$1, U$3: value POLOLUESTEPPERDRIVER -> 03-JST-B3B-XH-A; device reprap:DIL16 -> bt_con-jst-xh:B3B-XH
- moved U$7 183.1 mm to (116.8, 16.5), turned to 90 degrees
- moved U$8 177.9 mm to (90.2, 17.8), turned to 90 degrees
- moved U$3 137.1 mm to (-139.7, -110.5)
- moved U$1 135.2 mm to (-139.7, -100.3)
- moved U$6 126.8 mm to (64.8, -3.81), turned to 270 degrees
- moved U$2 115.9 mm to (35.6, 20.3)
Connections:
- removed net DIR_E3: U$8.9
- removed net DIR_Z1: U$4.9
- removed net DIR_Z2: U$5.9
- removed net END_X: U$9.P$2
- removed net END_Y: U$10.P$2
- removed net END_Z: U$11.P$2
- removed net N$10: U$1.11, U$1.12
- removed net N$24: JP6.1, U$3.13
- removed net N$25: JP6.3, U$3.14
- removed net N$26: JP6.5, R6.2, U$3.15
- removed net N$28: JP7.3, U$1.14
- removed net N$29: JP7.5, R7.2, U$1.15
- removed net N$57: U$3.3, X13.P$1, X6.P$1
- removed net N$58: U$3.4, X13.P$2, X6.P$2
- removed net N$59: U$3.5, X13.P$3, X6.P$3
- removed net N$60: U$3.6, X13.P$4, X6.P$4
- removed net N$61: U$1.3, X14.P$1, X7.P$1
- removed net N$62: U$1.4, X14.P$2, X7.P$2
- removed net N$63: U$1.5, X14.P$3, X7.P$3
- removed net N$64: U$1.6, X14.P$4, X7.P$4
- removed net N$67: Q3.2, X16.P$3, X16.P$4
- removed net N$9: U$3.11, U$3.12
- removed net Q_E3: Q3.1
- removed net STEP_E3: U$8.10
- removed net STEP_Z1: U$4.10
- removed net STEP_Z2: U$5.10
- removed net TRM_E3: C11.+, R8.1, U$16.P$2
- new net DIR_Z: U$2.PB5, U$6.9
- new net STEP_Z: U$2.PB4, U$6.10
- new net X+: U$2.PE3, U$9.P$2
- new net X-: U$10.P$2, U$2.PE4
- new net Y+: U$11.P$2, U$2.PE5
- new net Y-: U$1.P$2, U$2.PF4
- new net Z+: U$2.PF3, U$3.P$2
- new net Z-: U$12.P$2, U$2.PF2
- net +12V: no longer C6.+, C7.+, U$1.1, U$3.1, X16.P$1, X16.P$2
- net +5V: no longer JP6.2, JP6.4, JP6.6, JP7.2, JP7.4, JP7.6, R8.2, U$1.7, U$3.7
- net DIR_E1: now also U$2.PB3, U$7.9; no longer U$6.9
- net DIR_E2: now also U$2.PB1, U$8.9; no longer U$7.9
- net DIR_X: now also U$2.PD1, U$4.9; no longer U$1.9
- net DIR_Y: now also U$5.9; no longer U$3.9
- net GND: now also U$1.P$3, U$12.P$3, U$3.P$3; no longer C11.-, C6.-, C7.-, Q3.3, R6.1, R7.1, U$1.2, U$1.8, U$16.P$3, U$3.2, U$3.8
- net N$27: now also U$2.PB7; no longer JP7.1, U$1.13
- net N$37: no longer X8.P$1
- net N$38: no longer X8.P$2
- net N$39: no longer X8.P$3
- net N$40: no longer X8.P$4
- net N$41: no longer X9.P$1
- net N$42: no longer X9.P$2
- net N$43: no longer X9.P$3
- net N$44: no longer X9.P$4
- net N$49: no longer X11.P$1
- net N$50: no longer X11.P$2
- net N$51: no longer X11.P$3
- net N$52: no longer X11.P$4
- net N$53: no longer X12.P$1
- net N$54: no longer X12.P$2
- net N$55: no longer X12.P$3
- net N$56: no longer X12.P$4
- net N$66: now also U$1.P$1, U$12.P$1, U$3.P$1
- net Q_BED: now also U$2.PD2
- net Q_E1: now also U$2.PD3
- net Q_E2: now also U$2.PD6
- net STEP_E1: now also U$2.PB2, U$7.10; no longer U$6.10
- net STEP_E2: now also U$2.PB0, U$8.10; no longer U$7.10
- net STEP_EN: no longer U$1.16, U$3.16
- net STEP_X: now also U$2.PD0, U$4.10; no longer U$1.10
- net STEP_Y: now also U$2.PB6, U$5.10; no longer U$3.10
- net TRM_BED: now also U$2.PD7
- net TRM_E1: now also U$2.PF0
- net TRM_E2: now also U$2.PF1
