File: stellarcore/untitled.sch (EAGLE design)
At the start: 77 parts, among them Q3 IRF540, Q4 IRF540, Q5 IRF540, Q6 IRF540, X1 04-JST-B4B-XH-A, X10 04-JST-B4B-XH-A, X11 04-JST-B4B-XH-A, X12 04-JST-B4B-XH-A, X13 04-JST-B4B-XH-A, X14 04-JST-B4B-XH-A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

Commit message: new projects
Parts:
- removed C11: (no value), rcl:CPOL-EUE2.5-5
- removed C6, C7: (no value), rcl:CPOL-EUE2.5-7
- removed JP6, JP7: (no value), jumper:JP3Q
- removed Q3: IRF540, transistor-fet:IRF540
- removed R6, R7, R8: (no value), rcl:R-EU_0204/7
- removed U$16: 03-JST-B3B-XH-A, bt_con-jst-xh:03-JST-B3B-XH-A
- removed X11, X12, X13, X14, X16, X6, X7, X8, X9: 04-JST-B4B-XH-A, bt_con-jst-xh:04-JST-B4B-XH-A
- added U$12: 03-JST-B3B-XH-A, bt_con-jst-xh:03-JST-B3B-XH-A
- U$1, U$3: value POLOLUESTEPPERDRIVER -> 03-JST-B3B-XH-A; device reprap:POLOLUESTEPPERDRIVER -> bt_con-jst-xh:03-JST-B3B-XH-A
Connections:
- removed net DIR_E3: U$8.DIR
- removed net DIR_Z1: U$4.DIR
- removed net DIR_Z2: U$5.DIR
- removed net END_X: U$9-2.1
- removed net END_Y: U$10-2.1
- removed net END_Z: U$11-2.1
- removed net N$10: U$1.RST, U$1.SLP
- removed net N$24: JP6.1, U$3.MS3
- removed net N$25: JP6.3, U$3.MS2
- removed net N$26: JP6.5, R6.2, U$3.MS1
- removed net N$28: JP7.3, U$1.MS2
- removed net N$29: JP7.5, R7.2, U$1.MS1
- removed net N$57: U$3.2B, X13-1.1, X6-1.1
- removed net N$58: U$3.2A, X13-2.1, X6-2.1
- removed net N$59: U$3.1A, X13-3.1, X6-3.1
- removed net N$60: U$3.1B, X13-4.1, X6-4.1
- removed net N$61: U$1.2B, X14-1.1, X7-1.1
- removed net N$62: U$1.2A, X14-2.1, X7-2.1
- removed net N$63: U$1.1A, X14-3.1, X7-3.1
- removed net N$64: U$1.1B, X14-4.1, X7-4.1
- removed net N$67: Q3.D, X16-3.1, X16-4.1
- removed net N$9: U$3.RST, U$3.SLP
- removed net Q_E3: Q3.G
- removed net STEP_E3: U$8.STEP
- removed net STEP_Z1: U$4.STEP
- removed net STEP_Z2: U$5.STEP
- removed net TRM_E3: C11.+, R8.1, U$16-2.1
- new net DIR_Z: U$2.PB5, U$6.DIR
- new net STEP_Z: U$2.PB4, U$6.STEP
- new net X+: U$2.PE3, U$9-2.1
- new net X-: U$10-2.1, U$2.PE4
- new net Y+: U$11-2.1, U$2.PE5
- new net Y-: U$1-2.1, U$2.PF4
- new net Z+: U$2.PF3, U$3-2.1
- new net Z-: U$12-2.1, U$2.PF2
- net +12V: no longer C6.+, C7.+, U$1.VMOT, U$3.VMOT, X16-1.1, X16-2.1
- net +5V: no longer JP6.2, JP6.4, JP6.6, JP7.2, JP7.4, JP7.6, R8.2, U$1.VDD, U$3.VDD
- net DIR_E1: now also U$2.PB3, U$7.DIR; no longer U$6.DIR
- net DIR_E2: now also U$2.PB1, U$8.DIR; no longer U$7.DIR
- net DIR_X: now also U$2.PD1, U$4.DIR; no longer U$1.DIR
- net DIR_Y: now also U$5.DIR; no longer U$3.DIR
- net GND: now also U$1-3.1, U$12-3.1, U$3-3.1; no longer C11.-, C6.-, C7.-, Q3.S, R6.1, R7.1, U$1.GND1, U$1.GND2, U$16-3.1, U$3.GND1, U$3.GND2
- net N$27: now also U$2.PB7; no longer JP7.1, U$1.MS3
- net N$37: no longer X8-1.1
- net N$38: no longer X8-2.1
- net N$39: no longer X8-3.1
- net N$40: no longer X8-4.1
- net N$41: no longer X9-1.1
- net N$42: no longer X9-2.1
- net N$43: no longer X9-3.1
- net N$44: no longer X9-4.1
- net N$49: no longer X11-1.1
- net N$50: no longer X11-2.1
- net N$51: no longer X11-3.1
- net N$52: no longer X11-4.1
- net N$53: no longer X12-1.1
- net N$54: no longer X12-2.1
- net N$55: no longer X12-3.1
- net N$56: no longer X12-4.1
- net N$66: now also U$1-1.1, U$12-1.1, U$3-1.1
- net Q_BED: now also U$2.PD2
- net Q_E1: now also U$2.PD3
- net Q_E2: now also U$2.PD6
- net STEP_E1: now also U$2.PB2, U$7.STEP; no longer U$6.STEP
- net STEP_E2: now also U$2.PB0, U$8.STEP; no longer U$7.STEP
- net STEP_EN: no longer U$1.EN, U$3.EN
- net STEP_X: now also U$2.PD0, U$4.STEP; no longer U$1.STEP
- net STEP_Y: now also U$2.PB6, U$5.STEP; no longer U$3.STEP
- net TRM_BED: now also U$2.PD7
- net TRM_E1: now also U$2.PF0
- net TRM_E2: now also U$2.PF1
Other:
- moved on the sheet: C10, C8, C9, JP8, Q4, Q5, Q6, R11, R12, R9, U$10-1, U$10-2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
